File: ISE2024 PCB/ISE2024 kibann.sch (EAGLE design)
At the start: 52 parts, among them CN1 DM3AT, SW1 SRIDE_SWITCH

Commit message: Update ISE2024 kibann.sch
Connections:
- new net LED1.3: U$1.D14
- net +5V: no longer CON1.P$2, CON3.P$2
- net +5V_SV: now also CON1.P$2, CON3.P$2
- net BOARD-RX: now also U$1.D8; no longer U$1.D16
- net BOARD-TX: now also U$1.D9; no longer U$1.D15
- net LED1.0: now also U$1.D16; no longer U$1.D7
- net LED1.1: now also U$1.D15; no longer U$1.D8
- net LED1.2: no longer U$1.D9
Changed lines of the file:
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@@
 <part name="GND37" library="supply1" library_urn="urn:adsk.eagle:library:371" deviceset="GND" device=""/>
 <part name="CON1" library="XR Connector" library_urn="urn:adsk.eagle:library:38467597" deviceset="3PIN" device="" package3d_urn="urn:adsk.eagle:package:38467938/2"/>
-<part name="P+4" library="supply1" library_urn="urn:adsk.eagle:library:371" deviceset="+5V" device=""/>
 <part name="GND5" library="supply1" library_urn="urn:adsk.eagle:library:371" deviceset="GND" device=""/>
 <part name="CON3" library="XR Connector" library_urn="urn:adsk.eagle:library:38467597" deviceset="3PIN" device="" package3d_urn="urn:adsk.eagle:package:38467938/2"/>
-<part name="P+5" library="supply1" library_urn="urn:adsk.eagle:library:371" deviceset="+5V" device=""/>
 <part name="GND6" library="supply1" library_urn="urn:adsk.eagle:library:371" deviceset="GND" device=""/>
 <part name="GND26" library="supply1" library_urn="urn:adsk.eagle:library:371" deviceset="GND" device=""/>
@@
 <attribute name="NAME" x="-124.46" y="421.64" size="1.27" layer="95"/>
 </instance>
-<instance part="P+4" gate="1" x="-119.38" y="401.32" smashed="yes" rot="R180">
-<attribute name="VALUE" x="-116.84" y="406.4" size="1.778" layer="96" rot="R270"/>
-</instance>
 <instance part="GND5" gate="1" x="-111.76" y="401.32" smashed="yes">
 <attribute name="VALUE" x="-114.3" y="398.78" size="1.778" layer="96"/>
@@
 <instance part="CON3" gate="G$1" x="-149.86" y="416.56" smashed="yes">
 <attribute name="NAME" x="-152.4" y="421.64" size="1.27" layer="95"/>
-</instance>
-<instance part="P+5" gate="1" x="-147.32" y="401.32" smashed="yes" rot="R180">
-<attribute name="VALUE" x="-144.78" y="406.4" size="1.778" layer="96" rot="R270"/>
 </instance>
 <instance part="GND6" gate="1" x="-139.7" y="401.32" smashed="yes">
@@
 <pinref part="P+2" gate="1" pin="+5V"/>
 <pinref part="C2" gate="G$1" pin="1"/>
-</segment>
-<segment>
-<pinref part="CON1" gate="G$1" pin="P$2"/>
-<wire x1="-119.38" y1="414.02" x2="-119.38" y2="403.86" width="0.1524" layer="91"/>
-<pinref part="P+4" gate="1" pin="+5V"/>
-</segment>
-<segment>
-<pinref part="CON3" gate="G$1" pin="P$2"/>
-<wire x1="-147.32" y1="414.02" x2="-147.32" y2="403.86" width="0.1524" layer="91"/>
-<pinref part="P+5" gate="1" pin="+5V"/>
 </segment>
 <segment>
@@
 <net name="BOARD-RX" class="0">
 <segment>
-<pinref part="U$1" gate="G$1" pin="D16"/>
-<wire x1="-462.28" y1="353.06" x2="-459.74" y2="353.06" width="0.1524" layer="91"/>
-<label x="-459.74" y="353.06" size="1.778" layer="95" xref="yes"/>
-</segment>
-<segment>
 <pinref part="U$7" gate="G$1" pin="D16"/>
 <wire x1="-482.6" y1="119.38" x2="-490.22" y2="119.38" width="0.1524" layer="91"/>
 <label x="-490.22" y="119.38" size="1.778" layer="95" rot="R180" xref="yes"/>
 </segment>
+<segment>
+<pinref part="U$1" gate="G$1" pin="D8"/>
+<wire x1="-497.84" y1="347.98" x2="-500.38" y2="347.98" width="0.1524" layer="91"/>
+<label x="-500.38" y="347.98" size="1.778" layer="95" rot="R180" xref="yes"/>
+</segment>
 </net>
 <net name="BOARD-TX" class="0">
-<segment>
-<pinref part="U$1" gate="G$1" pin="D15"/>
-<wire x1="-462.28" y1="347.98" x2="-459.74" y2="347.98" width="0.1524" layer="91"/>
-<label x="-459.74" y="347.98" size="1.778" layer="95" xref="yes"/>
-</segment>
 <segment>
 <pinref part="U$7" gate="G$1" pin="D15"/>
@@
 <label x="-490.22" y="124.46" size="1.778" layer="95" rot="R180" xref="yes"/>
 </segment>
+<segment>
+<pinref part="U$1" gate="G$1" pin="D9"/>
+<wire x1="-497.84" y1="342.9" x2="-500.38" y2="342.9" width="0.1524" layer="91"/>
+<label x="-500.38" y="342.9" size="1.778" layer="95" rot="R180" xref="yes"/>
+</segment>
 </net>
 <net name="LED1.0" class="0">
-<segment>
-<pinref part="U$1" gate="G$1" pin="D7"/>
-<wire x1="-497.84" y1="353.06" x2="-500.38" y2="353.06" width="0.1524" layer="91"/>
-<label x="-500.38" y="353.06" size="1.778" layer="95" rot="R180" xref="yes"/>
-</segment>
 <segment>
 <pinref part="R13" gate="G$1" pin="2"/>
@@
 <label x="-408.94" y="307.34" size="1.778" layer="95" rot="R90" xref="yes"/>
 </segment>
+<segment>
+<pinref part="U$1" gate="G$1" pin="D16"/>
+<wire x1="-462.28" y1="353.06" x2="-454.66" y2="353.06" width="0.1524" layer="91"/>
+<label x="-454.66" y="353.06" size="1.778" layer="95" xref="yes"/>
+</segment>
 </net>
 <net name="LED1.1" class="0">
-<segment>
-<pinref part="U$1" gate="G$1" pin="D8"/>
-<wire x1="-497.84" y1="347.98" x2="-500.38" y2="347.98" width="0.1524" layer="91"/>
-<label x="-500.38" y="347.98" size="1.778" layer="95" rot="R180" xref="yes"/>
-</segment>
 <segment>
 <pinref part="R12" gate="G$1" pin="2"/>
@@
 <label x="-401.32" y="307.34" size="1.778" layer="95" rot="R90" xref="yes"/>
 </segment>
+<segment>
+<pinref part="U$1" gate="G$1" pin="D15"/>
+<wire x1="-462.28" y1="347.98" x2="-454.66" y2="347.98" width="0.1524" layer="91"/>
+<label x="-454.66" y="347.98" size="1.778" layer="95" xref="yes"/>
+</segment>
 </net>
 <net name="LED1.2" class="0">
-<segment>
-<pinref part="U$1" gate="G$1" pin="D9"/>
-<wire x1="-497.84" y1="342.9" x2="-500.38" y2="342.9" width="0.1524" layer="91"/>
-<label x="-500.38" y="342.9" size="1.778" layer="95" rot="R180" xref="yes"/>
-</segment>
 <segment>
 <pinref part="R11" gate="G$1" pin="2"/>
@@
 <pinref part="C4" gate="G$1" pin="1"/>
 <label x="-393.7" y="167.64" size="1.778" layer="95" xref="yes"/>
+</segment>
+<segment>
+<pinref part="CON3" gate="G$1" pin="P$2"/>
+<wire x1="-147.32" y1="414.02" x2="-147.32" y2="403.86" width="0.1524" layer="91"/>
+<label x="-147.32" y="403.86" size="1.778" layer="95" rot="R270" xref="yes"/>
+<label x="-147.32" y="403.86" size="1.778" layer="95" rot="R270" xref="yes"/>
+<label x="-147.32" y="403.86" size="1.778" layer="95" rot="R270" xref="yes"/>
+</segment>
+<segment>
+<pinref part="CON1" gate="G$1" pin="P$2"/>
+<wire x1="-119.38" y1="414.02" x2="-119.38" y2="403.86" width="0.1524" layer="91"/>
+<label x="-119.38" y="403.86" size="1.778" layer="95" rot="R270" xref="yes"/>
 </segment>
 </net>
@@
 </segment>
 </net>
+<net name="LED1.3" class="0">
+<segment>
+<pinref part="U$1" gate="G$1" pin="D14"/>
+<wire x1="-462.28" y1="342.9" x2="-454.66" y2="342.9" width="0.1524" layer="91"/>
+<label x="-454.66" y="342.9" size="1.778" layer="95" xref="yes"/>
+</segment>
+</net>
