File: NSE14/GPSsd1.1.sch (EAGLE design)
At the start: 34 parts, among them Q2 16mhz, SW1 SRIDE_SWITCH

Commit message: i
u
Parts:
- removed BMP1: BMP180, BMP180:BMP180
- removed BORD2, BORD3: (no value), PinSocket:2X10
- removed C1: 10uF, rcl:C-EU025-024X044
- removed C2, C3: 3.3uF, rcl:C-EU025-024X044
- removed C6, C7: 22p, rcl:C-EU025-024X044
- removed CON2, CON5: (no value), XR Connector:2PIN
- removed D1: 1N4148DO35-7, diode:1N4148DO35-7
- removed DCDC1: (no value), DC-DC:5V1A_M78AR05-1
- removed DCDC2: (no value), DC-DC:3.3V1A_M78AR033-1
- removed IM2: IM920_IM920C, CANSAT12th:IM920_IM920C
- removed Q2: 16mhz, crystal:CRYSTALHC49S
- removed SRIDE_SWTCH2, SW1: SRIDE_SWITCH, Sride Switch:SRIDE_SWITCH
- removed U$3: 2SK4017-NCH, mosfet:2SK4017-NCH
- removed U$4, U$5: 2SJ681-PCH, mosfet:2SJ681-PCH
- removed U$6: ATMEGA238P, atmega328p:ATMEGA238P
- added BMX2: BMX055, BMX055:BMX055
- added BORD1, BORD4: (no value), pinhead:PINHD-2X10/90
- added C4, C5: 22p, rcl:C-EU025-024X044
- added CN1: DM3AT, microSD:DM3AT
- added Q1: 16mhz, crystal:CRYSTALHC49S
- added R1, R11: (no value), rcl:R-US_0204/7
- added R14, R15: 10k, rcl:R-US_0204/7
- added R4: 100, rcl:R-US_0204/7
- added SRIDE_SWTCH1: SRIDE_SWITCH, Sride Switch:SRIDE_SWITCH
- added U$1: ATMEGA238P, atmega328p:ATMEGA238P
- R10, R8: value 1k -> (none)
- R12: value 100 -> (none)
- R2, R3: value (none) -> 10k
- R5: value 10k -> (none)
- R9: value 100k -> (none)
- U$2: value 2SJ681-PCH -> NEWGPS; device mosfet:2SJ681-PCH -> New_GPS:NEWGPS
Connections:
- removed net +5V1: DCDC1.VIN, U$5.DRAIN
- removed net FP: CON5.P$1, D1.A, R10.2, U$2.GATE, U$3.GATE, U$4.GATE
- removed net FP_CHECKER: C1.1, R8.2
- removed net IM_BUSY: IM2.BUSY/IO1, U$6.D6
- removed net IM_RESET: IM2.RESET, U$6.D5
- removed net LED: IM2.STATUS
- removed net N$1 (its old number): U$2.DRAIN, U$4.DRAIN
- removed net N$14: R7.2, R8.1, U$3.SOURCE
- removed net N$20: BORD3.P$17
- removed net RAW: CON2.P$2, U$2.SOURCE
- removed net RX_IM: IM2.RXD/IO6, U$6.D7
- removed net SW: R9.1, SW1.L, U$5.GATE
- removed net TX_IM: IM2.TXD/IO7, U$6.D8
- new net CLK: CN1.CLK, R6.1, U$1.SCKD13
- new net GPSRX: U$1.D7
- new net GPSTX: U$1.D8, U$2.RX, U$2.TX
- new net N$15: U$2.EN
- new net N$5: C5.1, Q1.1, U$1.PB7
- new net N$6: R1.2, SRIDE_SWTCH1.R, U$1.RESET
- new net N$7: C4.1, Q1.2, U$1.PB6
- new net N$9: BORD1.14, R11.1
- new net RST: U$1.D6, U$2.RST
- new net SD-MISO: CN1.DAT0, R7.1, U$1.MISOD12
- new net SD-MOSI: CN1.CMD, R3.1, U$1.MOSID11
- new net SD-SS: CN1.CD/DAT3, R2.1, U$1.SSD10
- net +3V3: now also BORD1.15, CN1.VDD, R14.1, R15.1, R2.2, R7.2; no longer BMP1.VIN, BORD2.P$10, BORD2.P$9, BORD3.P$15, BORD3.P$6, C3.1, DCDC2.VOUT, IM2.VCC, U$3.DRAIN
- net +5V: now also BMX2.VCC, BORD1.13, R1.1, R8.2, U$1.AVCC, U$1.VCC, U$2.5V; no longer BORD2.P$11, BORD2.P$12, BORD3.P$13, BORD3.P$8, C2.1, DCDC1.VOUT, DCDC2.VIN, R2.1, U$6.AVCC, U$6.VCC
- net BORDRX: now also BORD1.11, R9.2, U$1.D17; no longer BORD3.P$10, BORD3.P$11, U$6.D17
- net BORDTX: now also BORD1.9, R10.2, U$1.D16; no longer BORD3.P$12, BORD3.P$9, U$6.D16
- net GND: now also BMX2.GND, BORD1.5, C4.2, C5.2, CN1.VSS, R12.2, SRIDE_SWTCH1.LR, U$1.GND1, U$1.GND2, U$2.GND; no longer BMP1.GND, BORD2.P$13, BORD2.P$8, BORD3.P$16, BORD3.P$5, C1.2, C2.2, C3.2, C6.2, C7.2, CON2.P$1, CON5.P$2, DCDC1.GND, DCDC2.GND, IM2.GND, R10.1, R7.1, SRIDE_SWTCH2.LR, SW1.LR, U$6.GND1, U$6.GND2
- net LED1.0: now also U$1.D2; no longer U$6.D2
- net LED1.1: now also R4.2, U$1.D3; no longer R12.2, U$6.D3
- net N$10: now also BORD1.16; no longer LED4.A
- net N$11: now also LED4.A, R4.1; no longer BORD2.P$14
- net N$2: now also BORD1.6, R5.1; no longer C6.1, Q2.2, U$6.PB6
- net N$3: now also BORD1.8, R8.1; no longer D1.C, R9.2, U$4.SOURCE, U$5.SOURCE
- net N$4: now also BORD1.10, R9.1; no longer C7.1, Q2.1, U$6.PB7
- net N$8: now also BORD1.12, R10.1; no longer R2.2, SRIDE_SWTCH2.R, U$6.RESET
- net SCL: now also BMX2.SCL, R15.2, U$1.SCLD19; no longer BMP1.SCL, R6.1, U$6.SCLD19
- net SDA: now also BMX2.SDA, R14.2, U$1.SDAD18; no longer BMP1.SDA, R5.1, U$6.SDAD18
- net SERVO: now also BORD1.7, BORD4.10, BORD4.11, R11.2; no longer BORD3.P$14, BORD3.P$7, R3.1, U$6.D15
Other:
- note removed: "PWR"
- moved on the sheet: LED4, LED6, R10, R12, R13, R2, R3, R5, R6, R7, R8, R9
