File: NSE14/datalogger1.1.sch (EAGLE design)
At the start: 34 parts, among them Q2 16mhz, SW1 SRIDE_SWITCH

Commit message: i
u
Parts:
- removed BORD2, BORD3: (no value), PinSocket:2X10
- removed C1: 10uF, rcl:C-EU025-024X044
- removed C2, C3: 3.3uF, rcl:C-EU025-024X044
- removed CON2, CON5: (no value), XR Connector:2PIN
- removed D1: 1N4148DO35-7, diode:1N4148DO35-7
- removed DCDC1: (no value), DC-DC:5V1A_M78AR05-1
- removed DCDC2: (no value), DC-DC:3.3V1A_M78AR033-1
- removed IM2: IM920_IM920C, CANSAT12th:IM920_IM920C
- removed R10: 1k, rcl:R-US_0204/7
- removed SW1: SRIDE_SWITCH, Sride Switch:SRIDE_SWITCH
- removed U$2, U$4, U$5: 2SJ681-PCH, mosfet:2SJ681-PCH
- removed U$3: 2SK4017-NCH, mosfet:2SK4017-NCH
- added BMX1: BMX055, BMX055:BMX055
- added BORD1, BORD4: (no value), pinhead:PINHD-2X10/90
- added CN1: DM3AT, microSD:DM3AT
- added R1, R4: 10k, rcl:R-US_0204/7
- R3: value (none) -> 10k
- R8: value 1k -> 0
- R9: value 100k -> 0
Connections:
- removed net +5V1: DCDC1.VIN, U$5.DRAIN
- removed net BORDRX: BORD3.P$10, BORD3.P$11, U$6.D17
- removed net BORDTX: BORD3.P$12, BORD3.P$9, U$6.D16
- removed net FP: CON5.P$1, D1.A, R10.2, U$2.GATE, U$3.GATE, U$4.GATE
- removed net FP_CHECKER: C1.1, R8.2
- removed net IM_BUSY: IM2.BUSY/IO1, U$6.D6
- removed net IM_RESET: IM2.RESET, U$6.D5
- removed net LED: IM2.STATUS
- removed net N$1 (its old number): U$2.DRAIN, U$4.DRAIN
- removed net N$11: BORD2.P$14
- removed net N$14: R7.2, R8.1, U$3.SOURCE
- removed net N$20: BORD3.P$17
- removed net N$3: D1.C, R9.2, U$4.SOURCE, U$5.SOURCE
- removed net RAW: CON2.P$2, U$2.SOURCE
- removed net RX_IM: IM2.RXD/IO6, U$6.D7
- removed net SERVO: BORD3.P$14, BORD3.P$7, R3.1, U$6.D15
- removed net SW: R9.1, SW1.L, U$5.GATE
- removed net TX_IM: IM2.TXD/IO7, U$6.D8
- new net CLK: CN1.CLK, R6.1, U$6.SCKD13
- new net N$6: BORD1.10, R8.1
- new net N$9: BORD1.12, R9.1
- new net SD-MISO: CN1.DAT0, R7.1, U$6.MISOD12
- new net SD-MOSI: CN1.CMD, R3.1, U$6.MOSID11
- new net SD-SS: CN1.CD/DAT3, R1.1, U$6.SSD10
- net +3V3: now also BORD1.9, CN1.VDD, R1.2, R4.2, R7.2, R9.2; no longer BORD2.P$10, BORD2.P$9, BORD3.P$15, BORD3.P$6, C3.1, DCDC2.VOUT, IM2.VCC, U$3.DRAIN
- net +5V: now also BMX1.VCC, BORD1.11, R8.2; no longer BORD2.P$11, BORD2.P$12, BORD3.P$13, BORD3.P$8, C2.1, DCDC1.VOUT, DCDC2.VIN
- net GND: now also BMX1.GND, BORD1.13, BORD1.8, CN1.VSS; no longer BORD2.P$13, BORD2.P$8, BORD3.P$16, BORD3.P$5, C1.2, C2.2, C3.2, CON2.P$1, CON5.P$2, DCDC1.GND, DCDC2.GND, IM2.GND, R10.1, R7.1, SW1.LR
- net LED1.0: now also U$6.D7; no longer U$6.D2
- net LED1.1: now also U$6.D8; no longer U$6.D3
- net SCL: now also BMX1.SCL, R5.1; no longer R6.1
- net SDA: now also BMX1.SDA, R4.1; no longer R5.1
Other:
- note removed: "PWR"
- moved on the sheet: BMP1, C6, C7, LED4, LED6, Q2, R12, R13, R2, R3, R5, R6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
