File: NSE14/servodengen1.1.sch (EAGLE design)
At the start: 6 parts

Commit message: i
u
Parts:
- added D1: 1N4148DO35-7, diode:1N4148DO35-7
Connections:
- new net FP: D1.A
- net RAW: now also D1.C
Changed lines of the file:
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@@
 <part name="P+1" library="supply1" library_urn="urn:adsk.eagle:library:371" deviceset="+5V" device=""/>
 <part name="GND1" library="supply1" library_urn="urn:adsk.eagle:library:371" deviceset="GND" device=""/>
+<part name="D1" library="diode" library_urn="urn:adsk.eagle:library:210" deviceset="1N4148" device="DO35-7" package3d_urn="urn:adsk.eagle:package:43339/2"/>
 </parts>
 <sheets>
@@
 <instance part="GND1" gate="1" x="-12.7" y="7.62" smashed="yes">
 <attribute name="VALUE" x="-15.24" y="5.08" size="1.778" layer="96"/>
+</instance>
+<instance part="D1" gate="G$1" x="7.62" y="88.9" smashed="yes">
+<attribute name="NAME" x="10.16" y="89.3826" size="1.778" layer="95"/>
+<attribute name="VALUE" x="4.064" y="85.8266" size="1.27" layer="96"/>
 </instance>
 </instances>
@@
 <segment>
 <pinref part="DCDC1" gate="G$1" pin="VIN"/>
-<wire x1="25.4" y1="96.52" x2="25.4" y2="104.14" width="0.1524" layer="91"/>
-<wire x1="0" y1="96.52" x2="25.4" y2="96.52" width="0.1524" layer="91"/>
-<label x="0" y="96.52" size="1.778" layer="95" rot="R180" xref="yes"/>
+<label x="-2.54" y="88.9" size="1.778" layer="95" rot="R180" xref="yes"/>
+<wire x1="25.4" y1="104.14" x2="25.4" y2="88.9" width="0.1524" layer="91"/>
+<pinref part="D1" gate="G$1" pin="C"/>
+<wire x1="25.4" y1="88.9" x2="10.16" y2="88.9" width="0.1524" layer="91"/>
 </segment>
 </net>
@@
 </segment>
 </net>
+<net name="FP" class="0">
+<segment>
+<pinref part="D1" gate="G$1" pin="A"/>
+<wire x1="-2.54" y1="88.9" x2="5.08" y2="88.9" width="0.1524" layer="91"/>
+</segment>
+</net>
