File: NSE14ver2/SERVODENGEN ver2.sch (EAGLE design)
At the start: 7 parts

Commit message: 修正
Parts:
- removed D1: 1N4148DO35-7, diode:1N4148DO35-7
- added D2: (no value), ChipDiodes:1W4148W
Connections:
- net FP: now also D2.C; no longer D1.A
- net RAW: now also D2.A; no longer D1.C
Changed lines of the file:
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@@
 <part name="P+1" library="supply1" library_urn="urn:adsk.eagle:library:371" deviceset="+5V" device=""/>
 <part name="GND1" library="supply1" library_urn="urn:adsk.eagle:library:371" deviceset="GND" device=""/>
-<part name="D1" library="diode" library_urn="urn:adsk.eagle:library:210" deviceset="1N4148" device="DO35-7" package3d_urn="urn:adsk.eagle:package:43339/2"/>
+<part name="D2" library="ChipDiodes" library_urn="urn:adsk.eagle:library:42281194" deviceset="1W4148W" device="" package3d_urn="urn:adsk.eagle:package:42281200/2"/>
 </parts>
 <sheets>
@@
 <attribute name="VALUE" x="16.51" y="55.88" size="1.778" layer="96"/>
 </instance>
-<instance part="D1" gate="G$1" x="39.37" y="139.7" smashed="yes">
-<attribute name="NAME" x="41.91" y="140.1826" size="1.778" layer="95"/>
-<attribute name="VALUE" x="35.814" y="136.6266" size="1.27" layer="96"/>
+<instance part="D2" gate="G$1" x="40.64" y="139.7" smashed="yes" rot="R90">
+<attribute name="NAME" x="35.56" y="142.24" size="1.27" layer="95" rot="R90"/>
+<attribute name="VALUE" x="38.1" y="142.24" size="1.27" layer="96" rot="R90"/>
 </instance>
 </instances>
@@
 <label x="29.21" y="139.7" size="1.778" layer="95" rot="R180" xref="yes"/>
 <wire x1="57.15" y1="154.94" x2="57.15" y2="139.7" width="0.1524" layer="91"/>
-<pinref part="D1" gate="G$1" pin="C"/>
-<wire x1="57.15" y1="139.7" x2="41.91" y2="139.7" width="0.1524" layer="91"/>
+<wire x1="57.15" y1="139.7" x2="45.72" y2="139.7" width="0.1524" layer="91"/>
+<pinref part="D2" gate="G$1" pin="A"/>
 </segment>
 </net>
@@
 <net name="FP" class="0">
 <segment>
-<pinref part="D1" gate="G$1" pin="A"/>
-<wire x1="29.21" y1="139.7" x2="36.83" y2="139.7" width="0.1524" layer="91"/>
+<wire x1="29.21" y1="139.7" x2="35.56" y2="139.7" width="0.1524" layer="91"/>
+<pinref part="D2" gate="G$1" pin="C"/>
 </segment>
 </net>
