File: NSE14ver2/dengenver2.0.sch (EAGLE design)
At the start: 38 parts, among them Q1 16mhz, SW2 SRIDE_SWITCH

Commit message: 修正
Parts:
- removed D1: 1N4148DO35-7, diode:1N4148DO35-7
- removed LED4, LED6: (no value), led:LED5MM
- added D2: (no value), ChipDiodes:1W4148W
- added L1, L2: (no value), Chip LED:OSXX1608C1A
Connections:
- removed net N$1: C3.1, R1.2, SW1.P$2, U$1.PC6RESET
- new net RESETB: C3.1, JP1.6, R1.2, SW1.P$2, U$1.PC6RESET
- net +5V: now also R1.1
- net BORD1: now also BORD2.P$13, BORD2.P$8; no longer BORD2.P$16, BORD2.P$5, U$1.PB1
- net BORD2: now also BORD2.P$16, BORD2.P$5, U$1.PB1; no longer BORD2.P$13, BORD2.P$8, U$1.PD4
- net FP: now also D2.C; no longer D1.A
- net FP_CHECKER: now also U$1.PD4
- net GND: now also L1.CT, L2.CT; no longer LED4.C, LED6.C, R1.1
- net N$10: now also L1.AN; no longer LED4.A
- net N$3: now also D2.A; no longer D1.C
- net N$9: now also L2.AN; no longer LED6.A
- net SS: no longer JP1.6

Commit message: 328修正
Parts:
- U$1: device ATmega328p-PU:ATMEGA328P-AU -> ATMAGA328P-AU:ATMEGA328P-AU
Changed lines of the file:
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@@
 </classes>
 <parts>
-<part name="U$1" library="ATmega328p-PU" deviceset="ATMEGA328P-AU" device="" package3d_urn="urn:adsk.eagle:package:44716433/1"/>
+<part name="U$1" library="ATMAGA328P-AU" deviceset="ATMEGA328P-AU" device="" package3d_urn="urn:adsk.eagle:package:44744060/1"/>
 <part name="R1" library="rcl" library_urn="urn:adsk.eagle:library:334" deviceset="R-US_" device="R0603" package3d_urn="urn:adsk.eagle:package:23555/3" value="10k"/>
 <part name="Q1" library="crystal" library_urn="urn:adsk.eagle:library:204" deviceset="CRYSTAL" device="HC49UP" package3d_urn="urn:adsk.eagle:package:12078/1" value="16mhz"/>
