File: 14NSEver4/dataloggerver4.0.brd (EAGLE design)
At the start: 82.5 x 27.9 mm, 46 parts, among them CN1 DM3AT, CN2 DM3AT, Q1 16mhz, Q2 16mhz

Commit message: Completed board files ver1.0
Connections:
- new net 3V31: BMX2.3V3
- new net VCCIO1: BMX2.VCCIO
- net 3V3: no longer BMX2.3V3
- net VCCIO: no longer BMX2.VCCIO
Routing:
- net +3V3: track 100.8 -> 111.1 mm
Changed lines of the file:
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@@
 <signal name="VCCIO">
 <contactref element="BMX1" pad="VCCIO"/>
-<contactref element="BMX2" pad="VCCIO"/>
-<wire x1="7.7" y1="18.4" x2="17.86" y2="18.4" width="0" layer="19" extent="1-1"/>
 </signal>
 <signal name="3V3">
 <contactref element="BMX1" pad="3V3"/>
-<contactref element="BMX2" pad="3V3"/>
-<wire x1="7.7" y1="15.87" x2="17.86" y2="15.87" width="0" layer="19" extent="1-1"/>
 </signal>
 <signal name="+5V">
@@
 <contactref element="U$4" pad="5"/>
 <contactref element="U$6" pad="2"/>
+<via x="27.94" y="7.62" extent="1-16" drill="0.35"/>
+<via x="23.368" y="8.763" extent="1-16" drill="0.35"/>
+<via x="16.129" y="12.954" extent="1-16" drill="0.35"/>
+<via x="16.637" y="14.351" extent="1-16" drill="0.35"/>
+<via x="20.32" y="15.113" extent="1-16" drill="0.35"/>
+<via x="70.739" y="6.604" extent="1-16" drill="0.35"/>
+<via x="67.31" y="8.382" extent="1-16" drill="0.35"/>
+<via x="52.578" y="10.16" extent="1-16" drill="0.35"/>
+<via x="54.102" y="9.779" extent="1-16" drill="0.35"/>
+<via x="49.403" y="12.7" extent="1-16" drill="0.35"/>
+<via x="48.133" y="14.986" extent="1-16" drill="0.35"/>
+<via x="53.721" y="15.367" extent="1-16" drill="0.35"/>
+<via x="53.213" y="13.208" extent="1-16" drill="0.35"/>
+<via x="15.494" y="8.509" extent="1-16" drill="0.35"/>
+<via x="5.334" y="5.969" extent="1-16" drill="0.35"/>
+<via x="4.445" y="5.08" extent="1-16" drill="0.35"/>
+<via x="27.686" y="14.859" extent="1-16" drill="0.35"/>
+<via x="40.894" y="18.923" extent="1-16" drill="0.35"/>
+<via x="2.286" y="8.89" extent="1-16" drill="0.35"/>
+<via x="35.56" y="6.35" extent="1-16" drill="0.35"/>
+<via x="65.024" y="18.669" extent="1-16" drill="0.35"/>
+<via x="-0.254" y="20.32" extent="1-16" drill="0.35"/>
+<via x="-0.254" y="12.7" extent="1-16" drill="0.35"/>
+<via x="-0.254" y="6.35" extent="1-16" drill="0.35"/>
+<via x="16.256" y="0" extent="1-16" drill="0.35"/>
+<via x="4.826" y="1.27" extent="1-16" drill="0.35"/>
+<via x="12.446" y="17.78" extent="1-16" drill="0.35"/>
+<via x="9.906" y="10.16" extent="1-16" drill="0.35"/>
+<via x="28.956" y="17.78" extent="1-16" drill="0.35"/>
+<via x="50.546" y="25.4" extent="1-16" drill="0.35"/>
+<via x="8.509" y="25.654" extent="1-16" drill="0.35"/>
+<via x="20.066" y="25.654" extent="1-16" drill="0.35"/>
+<via x="63.246" y="-0.127" extent="1-16" drill="0.35"/>
+<via x="39.624" y="-0.127" extent="1-16" drill="0.35"/>
+<via x="75.438" y="0.381" extent="1-16" drill="0.35"/>
+<via x="79.502" y="6.604" extent="1-16" drill="0.35"/>
+<via x="80.264" y="11.938" extent="1-16" drill="0.35"/>
+<via x="80.01" y="20.447" extent="1-16" drill="0.35"/>
+<via x="73.406" y="24.892" extent="1-16" drill="0.35"/>
+<via x="70.358" y="19.05" extent="1-16" drill="0.35"/>
+<via x="72.898" y="16.256" extent="1-16" drill="0.35"/>
+<via x="36.068" y="12.192" extent="1-16" drill="0.35"/>
+<via x="58.293" y="10.541" extent="1-16" drill="0.35"/>
+<via x="61.214" y="12.573" extent="1-16" drill="0.35"/>
+<via x="45.466" y="25.4" extent="1-16" drill="0.35"/>
+<via x="44.196" y="19.05" extent="1-16" drill="0.35"/>
+<via x="69.596" y="25.4" extent="1-16" drill="0.35"/>
 </signal>
 <signal name="+3V3">
@@
 <wire x1="48.26" y1="21.17" x2="50.8" y2="21.17" width="0.3048" layer="1"/>
 <wire x1="48.26" y1="21.17" x2="45.72" y2="21.17" width="0.3048" layer="1"/>
-<wire x1="45.72" y1="21.17" x2="45.378" y2="21.17" width="0.3048" layer="1"/>
 <via x="45.72" y="21.17" extent="1-16" drill="0.35"/>
-<wire x1="41.91" y1="21.17" x2="45.72" y2="21.17" width="0.3048" layer="16"/>
 <wire x1="50.8" y1="21.17" x2="53.809" y2="21.17" width="0.3048" layer="1"/>
 <wire x1="26.25" y1="7.62" x2="26.25" y2="10.16" width="0.3048" layer="1"/>
@@
 <wire x1="5.969" y1="8.636" x2="5.969" y2="5.969" width="0.3048" layer="16"/>
 <wire x1="6.985" y1="4.953" x2="19.067" y2="4.953" width="0.3048" layer="16"/>
-<wire x1="63.5" y1="21.17" x2="63.5" y2="16.56" width="0" layer="19" extent="16-16"/>
-<wire x1="39.37" y1="16.56" x2="39.37" y2="21.17" width="0" layer="19" extent="16-16"/>
+<wire x1="39.37" y1="18.02486875" x2="39.37" y2="16.56" width="0.3048" layer="16"/>
+<wire x1="40.1994" y1="18.85426875" x2="39.37" y2="18.02486875" width="0.3048" layer="16"/>
+<wire x1="63.5" y1="21.17" x2="64.389" y2="20.281" width="0.3048" layer="16"/>
+<wire x1="64.389" y1="18.9113875" x2="63.5" y2="18.0223875" width="0.3048" layer="16"/>
+<wire x1="63.5" y1="18.0223875" x2="63.5" y2="16.56" width="0.3048" layer="16"/>
+<wire x1="64.389" y1="20.281" x2="64.389" y2="18.9113875" width="0.3048" layer="16"/>
+<wire x1="41.91" y1="21.17" x2="45.72" y2="21.17" width="0.3048" layer="16"/>
+<wire x1="39.37" y1="21.17" x2="40.1994" y2="20.3406" width="0.3048" layer="16"/>
+<wire x1="40.1994" y1="20.3406" x2="40.1994" y2="18.85426875" width="0.3048" layer="16"/>
 </signal>
 <signal name="SDA">
@@
 <wire x1="21.67" y1="7.43" x2="18.495" y2="7.43" width="0.3048" layer="16"/>
 <wire x1="18.495" y1="7.43" x2="17.098" y2="8.827" width="0.3048" layer="16"/>
-<wire x1="17.098" y1="11.303" x2="17.098" y2="8.827" width="0.3048" layer="16"/>
 <wire x1="24.55" y1="7.62" x2="24.36" y2="7.43" width="0.3048" layer="1"/>
 <wire x1="24.36" y1="7.43" x2="21.67" y2="7.43" width="0.3048" layer="1"/>
@@
 <wire x1="13.584" y1="15.87" x2="12.7" y2="14.986" width="0.3048" layer="16"/>
 <wire x1="12.7" y1="14.986" x2="12.7" y2="12.954" width="0.3048" layer="16"/>
-<wire x1="16.3487875" y1="12.0876" x2="17.098" y2="11.3383875" width="0.3048" layer="16"/>
+<wire x1="17.098" y1="11.3383875" x2="16.3487875" y2="12.0876" width="0.3048" layer="16"/>
 <wire x1="13.5664" y1="12.0876" x2="16.3487875" y2="12.0876" width="0.3048" layer="16"/>
 <wire x1="12.7" y1="12.954" x2="13.5664" y2="12.0876" width="0.3048" layer="16"/>
-<wire x1="17.098" y1="11.3383875" x2="17.098" y2="11.303" width="0" layer="19" extent="16-16"/>
+<wire x1="17.098" y1="8.827" x2="17.098" y2="11.3383875" width="0.3048" layer="16"/>
 </signal>
 <signal name="LED1.2">
@@
 <wire x1="34.329" y1="19.431" x2="35.306" y2="19.431" width="0.3048" layer="16"/>
 <via x="35.306" y="19.431" extent="1-16" drill="0.35"/>
-<wire x1="35.306" y1="19.431" x2="37.084" y2="19.431" width="0.3048" layer="1"/>
-<wire x1="38.36" y1="18.155" x2="38.36" y2="16.8813" width="0.3048" layer="1"/>
-<wire x1="37.084" y1="19.431" x2="38.36" y2="18.155" width="0.3048" layer="1"/>
+<wire x1="35.306" y1="19.431" x2="37.465" y2="19.431" width="0.3048" layer="1"/>
+<wire x1="37.725" y1="19.171" x2="37.725" y2="19.1673" width="0.3048" layer="1"/>
+<wire x1="38.36" y1="18.5323" x2="38.36" y2="16.8813" width="0.3048" layer="1"/>
+<wire x1="38.36" y1="18.5323" x2="37.725" y2="19.1673" width="0.3048" layer="1"/>
+<wire x1="37.465" y1="19.431" x2="37.725" y2="19.171" width="0.3048" layer="1"/>
 <via x="40.132" y="17.907" extent="1-16" drill="0.35"/>
 <wire x1="40.132" y1="17.907" x2="40.47" y2="17.569" width="0.3048" layer="16"/>
@@
 <wire x1="4.572" y1="17.78" x2="5.969" y2="16.383" width="0.3048" layer="1"/>
 <wire x1="5.969" y1="16.383" x2="5.969" y2="14.351" width="0.3048" layer="1"/>
-<wire x1="5.969" y1="14.351" x2="6.604" y2="13.716" width="0.3048" layer="1"/>
-<wire x1="6.604" y1="13.716" x2="13.43" y2="13.716" width="0.3048" layer="1"/>
-<wire x1="13.462" y1="13.716" x2="13.43" y2="13.716" width="0.3048" layer="1"/>
 <via x="13.43" y="13.716" extent="1-16" drill="0.35"/>
 <wire x1="13.43" y1="13.716" x2="19.84345625" y2="13.716" width="0.3048" layer="16"/>
@@
 <wire x1="27.432" y1="11.303" x2="30.3304" y2="8.4046" width="0.3048" layer="1"/>
 <wire x1="30.3304" y1="8.4046" x2="30.3304" y2="7.2732125" width="0.3048" layer="1"/>
+<wire x1="6.604" y1="13.716" x2="13.43" y2="13.716" width="0.3048" layer="1"/>
+<wire x1="5.969" y1="14.351" x2="6.604" y2="13.716" width="0.3048" layer="1"/>
 </signal>
 <signal name="BORDRX">
@@
 <contactref element="SW2" pad="P$2"/>
 <contactref element="U$7" pad="1"/>
-<wire x1="51.39513125" y1="11.43" x2="51.65" y2="11.43" width="0.3048" layer="1"/>
 <wire x1="51.65" y1="13.97" x2="51.65" y2="11.43" width="0.3048" layer="1"/>
 <wire x1="51.65" y1="13.97" x2="50.7928" y2="14.8272" width="0.3048" layer="1"/>
@@
 <contactref element="U$7" pad="4"/>
 <via x="59.436" y="19.431" extent="1-16" drill="0.35"/>
-<wire x1="62.49" y1="16.8813" x2="62.49" y2="18.1513" width="0.3048" layer="1"/>
-<wire x1="62.49" y1="18.1513" x2="61.2103" y2="19.431" width="0.3048" layer="1"/>
-<wire x1="61.2103" y1="19.431" x2="59.436" y2="19.431" width="0.3048" layer="1"/>
+<wire x1="62.49" y1="16.8813" x2="62.49" y2="18.5323" width="0.3048" layer="1"/>
+<wire x1="62.49" y1="18.5323" x2="61.5913" y2="19.431" width="0.3048" layer="1"/>
+<wire x1="61.5913" y1="19.431" x2="59.436" y2="19.431" width="0.3048" layer="1"/>
 <wire x1="59.436" y1="19.431" x2="58.459" y2="19.431" width="0.3048" layer="16"/>
 <wire x1="58.459" y1="19.431" x2="58.42" y2="19.47" width="0.3048" layer="16"/>
@@
 <wire x1="37.465" y1="20.32" x2="38.1" y2="19.685" width="0.3048" layer="16"/>
 <via x="38.1" y="19.685" extent="1-16" drill="0.35"/>
-<wire x1="38.1" y1="19.685" x2="39.3474" y2="18.4376" width="0.3048" layer="1"/>
-<wire x1="39.3474" y1="18.4376" x2="40.3517875" y2="18.4376" width="0.3048" layer="1"/>
-<wire x1="40.3517875" y1="18.4376" x2="43.18" y2="15.6093875" width="0.3048" layer="1"/>
+<wire x1="43.18" y1="15.6093875" x2="39.1043875" y2="19.685" width="0.3048" layer="1"/>
+<wire x1="38.1" y1="19.685" x2="39.1043875" y2="19.685" width="0.3048" layer="1"/>
 <wire x1="43.18" y1="15.6093875" x2="43.18" y2="12.827" width="0.3048" layer="1"/>
 <wire x1="43.18" y1="12.827" x2="43.7476" y2="12.2594" width="0.3048" layer="1"/>
@@
 <wire x1="43.7476" y1="12.2594" x2="47.3114" y2="12.2594" width="0.3048" layer="1"/>
 </signal>
+<signal name="VCCIO1">
+<contactref element="BMX2" pad="VCCIO"/>
+</signal>
+<signal name="3V31">
+<contactref element="BMX2" pad="3V3"/>
+</signal>
 </signals>
