File: 14NSEver4/dataloggerver4.0.sch (EAGLE design)
At the start: 46 parts, among them CN1 DM3AT, CN2 DM3AT, Q1 16mhz, Q2 16mhz

Commit message: changed board files
Connections:
- net GPSRX: now also JP6.4
- net GPSTX: no longer JP6.4
Changed lines of the file:
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@@
 </variantdefs>
 <classes>
-<class number="0" name="default" width="0.4064" drill="0">
+<class number="0" name="default" width="0" drill="0">
 </class>
 </classes>
@@
 <pinref part="U$3" gate="G$1" pin="PD6"/>
 </segment>
-</net>
-<net name="GPSTX" class="0">
-<segment>
-<wire x1="368.3" y1="101.6" x2="368.3" y2="93.98" width="0.1524" layer="91"/>
-<label x="368.3" y="93.98" size="1.778" layer="95" rot="R270" xref="yes"/>
-<pinref part="U$3" gate="G$1" pin="PD7"/>
-</segment>
-<segment>
-<label x="500.38" y="63.5" size="1.778" layer="95" rot="R270" xref="yes"/>
-<pinref part="JP6" gate="A" pin="3"/>
-<wire x1="500.38" y1="78.74" x2="500.38" y2="63.5" width="0.1524" layer="91"/>
-</segment>
 <segment>
 <wire x1="505.46" y1="68.58" x2="505.46" y2="63.5" width="0.1524" layer="91"/>
@@
 </segment>
 </net>
+<net name="GPSTX" class="0">
+<segment>
+<wire x1="368.3" y1="101.6" x2="368.3" y2="93.98" width="0.1524" layer="91"/>
+<label x="368.3" y="93.98" size="1.778" layer="95" rot="R270" xref="yes"/>
+<pinref part="U$3" gate="G$1" pin="PD7"/>
+</segment>
+<segment>
+<label x="500.38" y="63.5" size="1.778" layer="95" rot="R270" xref="yes"/>
+<pinref part="JP6" gate="A" pin="3"/>
+<wire x1="500.38" y1="78.74" x2="500.38" y2="63.5" width="0.1524" layer="91"/>
+</segment>
+</net>

Commit message: Changed board file
Parts:
- removed JP1, JP4, JP6: (no value), pinhead:PINHD-1X6
- removed JP3, JP5: (no value), pinhead:PINHD-1X5
- added U$2, U$5, U$6: 1X5, pin_socket:1X5
- added U$4, U$7: 1X61X6_2.5, pin_socket:1X61X6_2.5
Connections:
- removed net N$5: JP6.6
- net +3V3: now also JP2.4; no longer JP3.4
- net +5V: now also JP2.3, U$2.P$1, U$4.P$6, U$5.P$1, U$6.P$1, U$7.P$6; no longer JP1.1, JP2.1, JP3.3, JP4.1, JP5.1, JP6.1
- net BORD1: now also JP2.1; no longer JP3.1
- net BORD2: now also JP2.5; no longer JP3.5
- net GND: now also U$2.P$2, U$4.P$5, U$5.P$2, U$6.P$2, U$7.P$5; no longer JP1.2, JP3.2, JP4.2, JP5.2, JP6.2
- net GPSRX: now also U$6.P$4; no longer JP6.4
- net GPSTX: now also U$6.P$3; no longer JP6.3
- net MISO: now also U$4.P$2; no longer JP1.4
- net MISO1: now also U$7.P$2; no longer JP4.4
- net MOSI: now also U$4.P$3; no longer JP1.5
- net MOSI1: now also U$7.P$3; no longer JP4.5
- net RESET: now also U$2.P$3; no longer JP2.3
- net RESET1: now also U$5.P$3; no longer JP5.3
- net RESETB: now also U$4.P$1; no longer JP1.6
- net RESETB1: now also U$7.P$1; no longer JP4.6
- net RST: now also U$6.P$5; no longer JP6.5
- net RX: now also U$2.P$4; no longer JP2.4
- net RX1: now also U$5.P$4; no longer JP5.4
- net SCK: now also U$4.P$4; no longer JP1.3
- net SCK1: now also U$7.P$4; no longer JP4.3
- net TX: now also U$2.P$5; no longer JP2.5
- net TX1: now also U$5.P$5; no longer JP5.5
Other:
- moved on the sheet: JP2

Commit message: Completed board files ver1.0
Connections:
- new net 3V31: BMX2.3V3
- new net VCCIO1: BMX2.VCCIO
Changed lines of the file:
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@@
+</segment>
+</net>
+<net name="VCCIO1" class="0">
+<segment>
+<pinref part="BMX2" gate="G$1" pin="VCCIO"/>
+<wire x1="515.62" y1="177.8" x2="515.62" y2="176.53" width="0.1524" layer="91"/>
+<wire x1="515.62" y1="176.53" x2="504.19" y2="176.53" width="0.1524" layer="91"/>
+<label x="515.62" y="177.8" size="1.778" layer="95" xref="yes"/>
+</segment>
+</net>
+<net name="3V31" class="0">
+<segment>
+<pinref part="BMX2" gate="G$1" pin="3V3"/>
+<wire x1="504.19" y1="173.99" x2="504.19" y2="172.72" width="0.1524" layer="91"/>
+<wire x1="504.19" y1="172.72" x2="510.54" y2="172.72" width="0.1524" layer="91"/>
+<wire x1="513.08" y1="172.72" x2="510.54" y2="172.72" width="0.1524" layer="91"/>
+<label x="513.08" y="172.72" size="1.778" layer="95" xref="yes"/>
 </segment>
 </net>
