File: 14NSEver4/dengenver4.0.sch (EAGLE design)
At the start: 44 parts, among them Q1 16mhz, SW2 SRIDE_SWITCH

Commit message: Completed board files ver1.0
Parts:
- removed U$7, U$9: 1X5, PinSocket:1X5
- added U$1, U$11: 1X5, pin_socket:1X5
- U$6: device PinSocket:1X5 -> pin_socket:1X5
Connections:
- net +3V3: now also U$1.P$2, U$11.P$1; no longer U$6.P$2, U$7.P$1
- net +5V: now also U$1.P$3, U$11.P$2, U$6.P$1; no longer U$6.P$3, U$7.P$2, U$9.P$1
- net BORD1: now also U$1.P$5; no longer U$6.P$5
- net BORD2: now also U$1.P$1; no longer U$6.P$1
- net BORDRX: now also U$11.P$3; no longer U$7.P$3
- net BORDTX: now also U$11.P$4; no longer U$7.P$4
- net GND: now also U$1.P$4, U$11.P$5, U$6.P$2; no longer U$6.P$4, U$7.P$5, U$9.P$2
- net LED_1.1: now also U$8.ADC6
- net RESET: now also U$6.P$3; no longer U$9.P$3
- net RX: now also U$6.P$4; no longer U$9.P$4
- net TX: now also U$6.P$5; no longer U$9.P$5
