File: 14NSEver4/dengenver4.0.brd (EAGLE design)
At the start: 80 x 25.4 mm, 44 parts, among them Q1 16mhz, SW2 SRIDE_SWITCH

Commit message: Changed board file
Parts:
- removed JP1: (no value), pinhead:1X06
- removed JP2: (no value), pinhead:1X05
- added U$10: 1X61X6_2.5, pin_socket:HDRVR6W64P254_1X6_1564X250X865B
- added U$9: 1X5, PinSocket:1X5
- moved L2 37.4 mm to (45.7, 12.7)
- moved R13 32.1 mm to (41.9, 12.7), turned to 180 degrees
- moved C1 19.7 mm to (29.2, 20.3), turned to 0 degrees
- moved R11 17.0 mm to (45.7, 6.35), turned to 270 degrees
- moved R4 16.3 mm to (43.2, 6.35), turned to 270 degrees
- moved SW1 11.5 mm to (34.3, 10.2)
- moved C2 8.98 mm to (11.4, 21.6)
- moved R14 8.13 mm to (34.3, 6.35)
- moved R15 8.13 mm to (34.3, 3.81)
- moved Q1 5.24 mm to (20.3, 17.8), turned to 180 degrees
- moved C3 3.81 mm to (30.5, 15.2), turned to 180 degrees
- moved R12 2.84 mm to (-19.1, 14.0)
- moved R1 2.84 mm to (30.5, 17.8), turned to 0 degrees
- moved U$8 2.84 mm to (24.1, 10.2), turned to 270 degrees
Connections:
- net LED1.1 renamed LED_1.1
- removed net LED1.0: R13.2
- net +5V: now also U$10.1, U$9.P$1; no longer JP1.1, JP2.1
- net GND: now also U$10.2, U$9.P$2; no longer JP1.2, JP2.2
- net LED_1.0: now also R13.2
- net MISO: now also U$10.4; no longer JP1.4
- net MOSI: now also U$10.5; no longer JP1.5
- net RESET: now also U$9.P$3; no longer JP2.3
- net RESETB: now also U$10.6; no longer JP1.6
- net RX: now also U$9.P$4; no longer JP2.4
- net SCK: now also U$10.3; no longer JP1.3
- net TX: now also U$9.P$5; no longer JP2.5
Routing:
- net SERVO5V: track 0.00 -> 32.4 mm
- net FP: track 0.00 -> 23.0 mm
- net +5V1: track 0.00 -> 14.1 mm
- net +5V: track 27.7 -> 36.2 mm
- net N$2: track 0.00 -> 3.81 mm

Commit message: Completed board files ver1.0
Parts:
- removed U$7, U$9: 1X5, PinSocket:1X5
- added U$1, U$11: 1X5, pin_socket:HDRVR5W64P254_1X5_1310X250X865B
- U$6: device PinSocket:1X5 -> pin_socket:HDRVR5W64P254_1X5_1310X250X865B
- moved L1 54.3 mm to (31.8, 3.81)
- moved R12 48.1 mm to (27.9, 3.81), turned to 180 degrees
- moved U$6 29.2 mm to (27.9, 24.1), turned to 180 degrees
- moved R14 2.54 mm to (34.3, 8.89)
- moved R15 2.54 mm to (34.3, 6.35)
- moved SW1 2.54 mm to (34.3, 12.7)
- moved C5 1.80 mm to (35.6, 15.2)
- moved R7 1.80 mm to (35.6, 20.3)
- moved R8 1.80 mm to (35.6, 17.8)
- moved C4 1.27 mm to (58.4, 14.0), turned to 270 degrees
- moved U$10 1.27 mm to (30.5, 1.27)
- moved C1 1.27 mm to (30.5, 20.3)
- moved C6 1.27 mm to (53.3, 11.4), turned to 90 degrees
- flipped R11 to the bottom, turned to 90 degrees
- flipped R4 to the bottom, turned to 90 degrees
Connections:
- net +3V3: now also U$1.2, U$11.1; no longer U$6.P$2, U$7.P$1
- net +5V: now also U$1.3, U$11.2, U$6.1; no longer U$6.P$3, U$7.P$2, U$9.P$1
- net BORD1: now also U$1.5; no longer U$6.P$5
- net BORD2: now also U$1.1; no longer U$6.P$1
- net BORDRX: now also U$11.3; no longer U$7.P$3
- net BORDTX: now also U$11.4; no longer U$7.P$4
- net GND: now also U$1.4, U$11.5, U$6.2; no longer U$6.P$4, U$7.P$5, U$9.P$2
- net LED_1.1: now also U$8.ADC6
- net RESET: now also U$6.3; no longer U$9.P$3
- net RX: now also U$6.4; no longer U$9.P$4
- net TX: now also U$6.5; no longer U$9.P$5
Routing:
- net +3V3: track 0.00 -> 129.2 mm, vias 0 -> 1
- net +5V: track 36.2 -> 138.1 mm, vias 0 -> 5
- net BORDRX: track 0.00 -> 57.1 mm, vias 0 -> 1
- net BORDTX: track 0.00 -> 56.8 mm, vias 0 -> 1
- net SERVO1: track 0.00 -> 48.4 mm
- net SERVO2: track 0.00 -> 34.2 mm, vias 0 -> 2
- net RESETB: track 0.00 -> 29.5 mm, vias 0 -> 2
- net N$3: track 0.00 -> 27.0 mm, vias 0 -> 1
- net BORD1: track 0.00 -> 26.9 mm, vias 0 -> 1
- net SCL: track 0.00 -> 26.5 mm, vias 0 -> 2
- net SDA: track 0.00 -> 22.5 mm, vias 0 -> 1
- net TX: track 0.00 -> 18.0 mm, vias 0 -> 1
- net BORD2: track 0.00 -> 17.0 mm
- net RX: track 0.00 -> 16.9 mm, vias 0 -> 1
- net IM_RESET: track 0.00 -> 16.3 mm, vias 0 -> 1
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Other:
- board size 80 x 25.4 mm -> 82.5 x 27.9 mm

Commit message: ver1.1 uploaded
Parts:
- moved U$10 1.27 mm to (30.5, 0.00)
- moved SW2 0.85 mm to (60.5, 4.70)
- moved U$2 0.76 mm to (48.3, 22.4)
- moved U$3 0.76 mm to (40.6, 22.4)
- moved U$4 0.76 mm to (44.5, 22.4)
- moved U$5 0.65 mm to (50.7, 3.17)
Routing:
- net +5V: track 138.1 -> 139.8 mm
- net +3V3: track 129.2 -> 130.5 mm
- net MOSI: track 9.23 -> 10.5 mm
- net RESETB: track 29.5 -> 30.8 mm
- net N$3: track 27.0 -> 27.9 mm
- net MISO: track 7.67 -> 8.57 mm
- net RAW: track 14.7 -> 15.5 mm
- net +5V1: track 14.1 -> 14.8 mm
- net SCK: track 7.29 -> 7.81 mm
- net SERVO2: track 34.2 -> 34.7 mm

Commit message: ver1.2
Parts:
- moved C2 5.24 mm to (10.2, 16.5)
- moved U$10 1.27 mm to (30.5, 1.27)
- moved IM2 1.27 mm to (22.9, 12.7)
Routing:
- net +5V: track 139.8 -> 138.0 mm
- net +3V3: track 130.5 -> 132.1 mm
- net MOSI: track 10.5 -> 9.23 mm
- net RESETB: track 30.8 -> 29.5 mm
- net MISO: track 8.57 -> 7.74 mm
- net RX_IM: track 7.75 -> 7.22 mm
- net IM_RESET: track 16.3 -> 15.8 mm

Commit message: changed board files
Parts:
- moved U$11 1.27 mm to (77.5, 17.8)
Routing:
- net BORDTX: track 56.8 -> 58.1 mm
- net BORDRX: track 57.1 -> 58.3 mm
- net +5V: track 138.0 -> 139.3 mm
- net +3V3: track 132.1 -> 133.3 mm
Other:
- board size 82.5 x 27.9 mm -> 83.8 x 27.9 mm
Changed lines of the file:
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@@
 <plain>
 <wire x1="-1.27" y1="-1.27" x2="-1.27" y2="26.67" width="0.0762" layer="20"/>
-<wire x1="-1.27" y1="26.67" x2="81.28" y2="26.67" width="0.0762" layer="20"/>
-<wire x1="81.28" y1="26.67" x2="81.28" y2="-1.27" width="0.0762" layer="20"/>
-<wire x1="81.28" y1="-1.27" x2="-1.27" y2="-1.27" width="0.0762" layer="20"/>
+<wire x1="-1.27" y1="26.67" x2="82.55" y2="26.67" width="0.0762" layer="20"/>
+<wire x1="82.55" y1="26.67" x2="82.55" y2="-1.27" width="0.0762" layer="20"/>
+<wire x1="82.55" y1="-1.27" x2="-1.27" y2="-1.27" width="0.0762" layer="20"/>
 <hole x="2.54" y="22.86" drill="3"/>
 <hole x="2.54" y="2.54" drill="3"/>
-<hole x="77.47" y="2.54" drill="3"/>
-<hole x="77.47" y="22.86" drill="3"/>
+<hole x="78.74" y="2.54" drill="3"/>
+<hole x="78.74" y="22.86" drill="3"/>
 </plain>
 <attributes>
@@
 <attribute name="VALUE" x="5.77" y="7.62" size="1.27" layer="27" rot="R90" align="top-center"/>
 </element>
-<element name="U$11" library="pin_socket" package="HDRVR5W64P254_1X5_1310X250X865B" package3d_urn="urn:adsk.eagle:package:44791100/1" value="1X5" x="76.2" y="17.78" smashed="yes" rot="R270">
-<attribute name="NAME" x="78.839" y="17.78" size="1.27" layer="25" rot="R270" align="bottom-center"/>
-<attribute name="VALUE" x="74.24" y="17.78" size="1.27" layer="27" rot="R270" align="top-center"/>
+<element name="U$11" library="pin_socket" package="HDRVR5W64P254_1X5_1310X250X865B" package3d_urn="urn:adsk.eagle:package:44791100/1" value="1X5" x="77.47" y="17.78" smashed="yes" rot="R270">
+<attribute name="NAME" x="80.109" y="17.78" size="1.27" layer="25" rot="R270" align="bottom-center"/>
+<attribute name="VALUE" x="75.51" y="17.78" size="1.27" layer="27" rot="R270" align="top-center"/>
 </element>
 <element name="U$6" library="pin_socket" package="HDRVR5W64P254_1X5_1310X250X865B" package3d_urn="urn:adsk.eagle:package:44791100/1" value="1X5" x="27.94" y="24.13" smashed="yes" rot="R180">
@@
 <wire x1="29.01779375" y1="2.64559375" x2="30.39339375" y2="1.26999375" width="0.508" layer="1"/>
 <wire x1="32.6" y1="1.27" x2="30.48" y2="1.27" width="0.508" layer="1"/>
-<wire x1="76.2" y1="15.24" x2="70.7388125" y2="15.24" width="0.508" layer="1"/>
+<wire x1="77.47" y1="15.24" x2="70.7388125" y2="15.24" width="0.508" layer="1"/>
 <wire x1="49.53" y1="15.24" x2="58" y2="15.24" width="0.508" layer="16"/>
 <wire x1="58" y1="15.24" x2="58.42" y2="14.82" width="0.508" layer="16"/>
@@
 <wire x1="8.81486875" y1="6.95" x2="8.1996" y2="6.33473125" width="0.3048" layer="16"/>
 <wire x1="46.1560375" y1="15.6760375" x2="47.862075" y2="13.97" width="0.3048" layer="16"/>
-<wire x1="76.2" y1="17.78" x2="52.07" y2="17.78" width="0.3048" layer="16"/>
+<wire x1="77.47" y1="17.78" x2="52.07" y2="17.78" width="0.3048" layer="16"/>
 <wire x1="52.07" y1="17.78" x2="48.768" y2="21.082" width="0.3048" layer="16"/>
 <wire x1="48.768" y1="21.082" x2="42.418" y2="21.082" width="0.3048" layer="16"/>
@@
 <wire x1="52.89473125" y1="8.6896" x2="56.27013125" y2="12.065" width="0.3048" layer="16"/>
 <wire x1="58.93565625" y1="12.065" x2="60.78705625" y2="13.9164" width="0.3048" layer="16"/>
-<wire x1="76.2" y1="12.7" x2="74.9836" y2="13.9164" width="0.3048" layer="16"/>
-<wire x1="74.9836" y1="13.9164" x2="60.78705625" y2="13.9164" width="0.3048" layer="16"/>
+<wire x1="77.47" y1="12.7" x2="76.2536" y2="13.9164" width="0.3048" layer="16"/>
+<wire x1="76.2536" y1="13.9164" x2="60.78705625" y2="13.9164" width="0.3048" layer="16"/>
 <wire x1="56.27013125" y1="12.065" x2="58.93565625" y2="12.065" width="0.3048" layer="16"/>
 </signal>
@@
 <wire x1="47.879" y1="8.763" x2="49.022" y2="7.62" width="0.3048" layer="16"/>
 <wire x1="49.022" y1="7.62" x2="53.34" y2="7.62" width="0.3048" layer="16"/>
-<wire x1="74.93" y1="11.43" x2="76.2" y2="10.16" width="0.3048" layer="16"/>
+<wire x1="76.2" y1="11.43" x2="77.47" y2="10.16" width="0.3048" layer="16"/>
 <wire x1="53.34" y1="7.62" x2="57.15" y2="11.43" width="0.3048" layer="16"/>
-<wire x1="57.15" y1="11.43" x2="74.93" y2="11.43" width="0.3048" layer="16"/>
+<wire x1="57.15" y1="11.43" x2="76.2" y2="11.43" width="0.3048" layer="16"/>
 </signal>
 <signal name="LED_1.1">
