File: 14NSEver4/dataloggerver4.1.sch (EAGLE design)
At the start: 46 parts, among them CN1 DM3AT, CN2 DM3AT, Q1 16mhz, Q2 16mhz

Commit message: changed v4.2
Parts:
- removed Q1, Q2: 16mhz, crystal:CRYSTALHC49UP
- added U$3, U$9: FE-238, FA-238:FE-238
Connections:
- net GND: now also U$3.GND, U$3.GND1, U$9.GND, U$9.GND1
- net N$14: now also U$9.3; no longer Q2.2
- net N$16: now also U$3.1; no longer Q1.1
- net N$17: now also U$3.3; no longer Q1.2
- net N$3: now also U$9.1; no longer Q2.1
Changed lines of the file:
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@@
 <part name="R13" library="rcl" library_urn="urn:adsk.eagle:library:334" deviceset="R-US_" device="R0603" package3d_urn="urn:adsk.eagle:package:23555/3" value="100"/>
 <part name="R10" library="rcl" library_urn="urn:adsk.eagle:library:334" deviceset="R-US_" device="R0603" package3d_urn="urn:adsk.eagle:package:23555/3" value="10k"/>
-<part name="Q1" library="crystal" library_urn="urn:adsk.eagle:library:204" deviceset="CRYSTAL" device="HC49UP" package3d_urn="urn:adsk.eagle:package:12078/1" value="16mhz"/>
 <part name="C1" library="rcl" library_urn="urn:adsk.eagle:library:334" deviceset="C-US" device="C1608" package3d_urn="urn:adsk.eagle:package:23621/2" value="22p"/>
 <part name="C2" library="rcl" library_urn="urn:adsk.eagle:library:334" deviceset="C-US" device="C1608" package3d_urn="urn:adsk.eagle:package:23621/2" value="22p"/>
@@
 <part name="GND8" library="supply1" library_urn="urn:adsk.eagle:library:371" deviceset="GND" device=""/>
 <part name="R16" library="rcl" library_urn="urn:adsk.eagle:library:334" deviceset="R-US_" device="R0603" package3d_urn="urn:adsk.eagle:package:23555/3" value="10k"/>
-<part name="Q2" library="crystal" library_urn="urn:adsk.eagle:library:204" deviceset="CRYSTAL" device="HC49UP" package3d_urn="urn:adsk.eagle:package:12078/1" value="16mhz"/>
 <part name="C4" library="rcl" library_urn="urn:adsk.eagle:library:334" deviceset="C-US" device="C1608" package3d_urn="urn:adsk.eagle:package:23621/2" value="22p"/>
 <part name="C5" library="rcl" library_urn="urn:adsk.eagle:library:334" deviceset="C-US" device="C1608" package3d_urn="urn:adsk.eagle:package:23621/2" value="22p"/>
@@
 <part name="GND14" library="supply1" library_urn="urn:adsk.eagle:library:371" deviceset="GND" device=""/>
 <part name="GND15" library="supply1" library_urn="urn:adsk.eagle:library:371" deviceset="GND" device=""/>
+<part name="U$3" library="FA-238" library_urn="urn:adsk.eagle:library:44894307" deviceset="FE-238" device="" package3d_urn="urn:adsk.eagle:package:44894250/2"/>
+<part name="GND17" library="supply1" library_urn="urn:adsk.eagle:library:371" deviceset="GND" device=""/>
+<part name="U$9" library="FA-238" library_urn="urn:adsk.eagle:library:44894307" deviceset="FE-238" device="" package3d_urn="urn:adsk.eagle:package:44894250/2"/>
+<part name="GND18" library="supply1" library_urn="urn:adsk.eagle:library:371" deviceset="GND" device=""/>
 </parts>
 <sheets>
@@
 <attribute name="VALUE" x="-15.24" y="147.828" size="1.778" layer="96"/>
 </instance>
-<instance part="Q1" gate="G$1" x="-3.81" y="105.41" smashed="yes" rot="R270">
-<attribute name="NAME" x="-2.794" y="102.87" size="1.778" layer="95" rot="R270"/>
-<attribute name="VALUE" x="-6.35" y="102.87" size="1.778" layer="96" rot="R270"/>
-</instance>
 <instance part="C1" gate="G$1" x="-13.97" y="107.95" smashed="yes" rot="R270">
 <attribute name="NAME" x="-13.335" y="106.934" size="1.778" layer="95" rot="R270"/>
@@
 <attribute name="VALUE" x="295.91" y="154.178" size="1.778" layer="96"/>
 </instance>
-<instance part="Q2" gate="G$1" x="314.96" y="99.06" smashed="yes" rot="R270">
-<attribute name="NAME" x="315.976" y="96.52" size="1.778" layer="95" rot="R270"/>
-<attribute name="VALUE" x="312.42" y="96.52" size="1.778" layer="96" rot="R270"/>
-</instance>
 <instance part="C4" gate="G$1" x="304.8" y="101.6" smashed="yes" rot="R270">
 <attribute name="NAME" x="305.435" y="100.584" size="1.778" layer="95" rot="R270"/>
@@
 <instance part="GND15" gate="1" x="119.38" y="68.58" smashed="yes">
 <attribute name="VALUE" x="116.84" y="66.04" size="1.778" layer="96"/>
+</instance>
+<instance part="U$3" gate="G$1" x="-5.08" y="104.14" smashed="yes">
+<attribute name="NAME" x="-7.62" y="110.236" size="1.778" layer="95"/>
+<attribute name="VALUE" x="-7.62" y="107.95" size="1.778" layer="96"/>
+</instance>
+<instance part="GND17" gate="1" x="-2.54" y="88.9" smashed="yes">
+<attribute name="VALUE" x="-5.08" y="86.36" size="1.778" layer="96"/>
+</instance>
+<instance part="U$9" gate="G$1" x="312.42" y="99.06" smashed="yes">
+<attribute name="NAME" x="309.88" y="105.156" size="1.778" layer="95"/>
+<attribute name="VALUE" x="309.88" y="102.87" size="1.778" layer="96"/>
+</instance>
+<instance part="GND18" gate="1" x="312.42" y="86.36" smashed="yes">
+<attribute name="VALUE" x="309.88" y="83.82" size="1.778" layer="96"/>
 </instance>
 </instances>
@@
 <wire x1="119.92" y1="77.47" x2="119.92" y2="79.82" width="0.1524" layer="91"/>
 <pinref part="GND15" gate="1" pin="GND"/>
+</segment>
+<segment>
+<pinref part="U$3" gate="G$1" pin="GND"/>
+<wire x1="-5.08" y1="99.06" x2="-5.08" y2="93.98" width="0.1524" layer="91"/>
+<wire x1="-5.08" y1="93.98" x2="-2.54" y2="93.98" width="0.1524" layer="91"/>
+<pinref part="U$3" gate="G$1" pin="GND1"/>
+<wire x1="-2.54" y1="93.98" x2="-2.54" y2="99.06" width="0.1524" layer="91"/>
+<wire x1="-2.54" y1="93.98" x2="-2.54" y2="91.44" width="0.1524" layer="91"/>
+<junction x="-2.54" y="93.98"/>
+<pinref part="GND17" gate="1" pin="GND"/>
+</segment>
+<segment>
+<pinref part="U$9" gate="G$1" pin="GND1"/>
+<wire x1="314.96" y1="93.98" x2="314.96" y2="91.44" width="0.1524" layer="91"/>
+<wire x1="314.96" y1="91.44" x2="312.42" y2="91.44" width="0.1524" layer="91"/>
+<pinref part="U$9" gate="G$1" pin="GND"/>
+<wire x1="312.42" y1="91.44" x2="312.42" y2="93.98" width="0.1524" layer="91"/>
+<wire x1="312.42" y1="88.9" x2="312.42" y2="91.44" width="0.1524" layer="91"/>
+<junction x="312.42" y="91.44"/>
+<pinref part="GND18" gate="1" pin="GND"/>
 </segment>
 </net>
@@
 <net name="N$3" class="0">
 <segment>
-<pinref part="Q2" gate="G$1" pin="1"/>
-<wire x1="314.96" y1="101.6" x2="307.34" y2="101.6" width="0.1524" layer="91"/>
-<junction x="314.96" y="101.6"/>
 <pinref part="C4" gate="G$1" pin="1"/>
 <pinref part="U$1" gate="G$1" pin="PB6"/>
-<wire x1="322.58" y1="101.6" x2="314.96" y2="101.6" width="0.1524" layer="91"/>
+<wire x1="309.88" y1="101.6" x2="307.34" y2="101.6" width="0.1524" layer="91"/>
+<wire x1="322.58" y1="101.6" x2="309.88" y2="101.6" width="0.1524" layer="91"/>
+<pinref part="U$9" gate="G$1" pin="1"/>
+<wire x1="309.88" y1="99.06" x2="309.88" y2="101.6" width="0.1524" layer="91"/>
+<junction x="309.88" y="101.6"/>
 </segment>
 </net>
 <net name="N$14" class="0">
 <segment>
-<pinref part="Q2" gate="G$1" pin="2"/>
-<wire x1="314.96" y1="96.52" x2="307.34" y2="96.52" width="0.1524" layer="91"/>
-<junction x="314.96" y="96.52"/>
+<wire x1="317.5" y1="96.52" x2="307.34" y2="96.52" width="0.1524" layer="91"/>
 <pinref part="C5" gate="G$1" pin="1"/>
 <pinref part="U$1" gate="G$1" pin="PB7"/>
 <wire x1="322.58" y1="99.06" x2="320.04" y2="99.06" width="0.1524" layer="91"/>
 <wire x1="320.04" y1="99.06" x2="320.04" y2="96.52" width="0.1524" layer="91"/>
-<wire x1="320.04" y1="96.52" x2="314.96" y2="96.52" width="0.1524" layer="91"/>
+<wire x1="320.04" y1="96.52" x2="317.5" y2="96.52" width="0.1524" layer="91"/>
+<pinref part="U$9" gate="G$1" pin="3"/>
+<wire x1="317.5" y1="99.06" x2="317.5" y2="96.52" width="0.1524" layer="91"/>
+<junction x="317.5" y="96.52"/>
 </segment>
 </net>
@@
 <pinref part="U$8" gate="G$1" pin="PB6"/>
 <wire x1="2.54" y1="106.68" x2="12.7" y2="106.68" width="0.1524" layer="91"/>
-<pinref part="Q1" gate="G$1" pin="1"/>
-<wire x1="-3.81" y1="107.95" x2="-11.43" y2="107.95" width="0.1524" layer="91"/>
-<junction x="-3.81" y="107.95"/>
 <pinref part="C1" gate="G$1" pin="1"/>
+<wire x1="-7.62" y1="107.95" x2="-11.43" y2="107.95" width="0.1524" layer="91"/>
 <wire x1="2.54" y1="106.68" x2="2.54" y2="107.95" width="0.1524" layer="91"/>
-<wire x1="2.54" y1="107.95" x2="-3.81" y2="107.95" width="0.1524" layer="91"/>
+<wire x1="2.54" y1="107.95" x2="-7.62" y2="107.95" width="0.1524" layer="91"/>
+<pinref part="U$3" gate="G$1" pin="1"/>
+<wire x1="-7.62" y1="104.14" x2="-7.62" y2="107.95" width="0.1524" layer="91"/>
+<junction x="-7.62" y="107.95"/>
 </segment>
 </net>
@@
 <pinref part="U$8" gate="G$1" pin="PB7"/>
 <wire x1="2.54" y1="104.14" x2="12.7" y2="104.14" width="0.1524" layer="91"/>
-<pinref part="Q1" gate="G$1" pin="2"/>
-<wire x1="-3.81" y1="102.87" x2="-11.43" y2="102.87" width="0.1524" layer="91"/>
-<junction x="-3.81" y="102.87"/>
+<wire x1="0" y1="102.87" x2="-11.43" y2="102.87" width="0.1524" layer="91"/>
 <pinref part="C2" gate="G$1" pin="1"/>
 <wire x1="2.54" y1="104.14" x2="2.54" y2="102.87" width="0.1524" layer="91"/>
-<wire x1="2.54" y1="102.87" x2="-3.81" y2="102.87" width="0.1524" layer="91"/>
-</segment>
-</net>
+<wire x1="2.54" y1="102.87" x2="0" y2="102.87" width="0.1524" layer="91"/>
+<pinref part="U$3" gate="G$1" pin="3"/>
+<wire x1="0" y1="104.14" x2="0" y2="102.87" width="0.1524" layer="91"/>
+<junction x="0" y="102.87"/>
+</segment>
+</net>
